File: KiCad 9 6502 ROR Test Board V2.0S/KiCad 9 6502 ROR Test Board V2.0S.kicad_pcb (KiCad board)
At the start: 2 copper layers, 55.6 x 153.4 mm, 28 parts, among them P1 CONN-TH_2P-P5.00, Q1 2N7002, Q2 2N7002, U1 6502, U2 AT28C256, U3 SN74HCT14DR, U4 SN74HCS74DR, U5 Plated Through Hole M3, U6 Plated Through Hole M3, U7 Plated Through Hole M3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

Commit message: added 3D models to KiCad
Added 3D Models of components to both KiCad Boards

Fixed footprint of screw terminal to match with 30.702 on both easyeda and kicad files

re-rendered 2D view from EasyEDA and  added 3D view rendering from KiCad

Renders in separate folder

Exported new gerbers from both EasyEDA and KiCad with updated footprint

Exported 3D model of both boards from KiCad and added to folder.

Updated link to smd LED to active part.
Connections:
- C5 pad 1: Net-(U3-6A) -> R4_1
